File: juno-chorus-clone.kicad_pcb (KiCad board)
At the start: 2 copper layers, 149.9 x 101.6 mm, 172 parts, among them P1 15VAC_IN, P2 AUDIO_IN, P3 AUDIO_OUT_1, P4 AUDIO_OUT_2, Q1 2SC1815, Q10 2SC1815, Q11 2SA1015, Q12 2SA1015, Q13 2SC1815, Q14 2SA1015, Q15 2SA1015, Q16 2SK30, Q17 2SK30, Q18 2SA1015, Q19 2SA1015, Q2 2SC1815, Q3 2SA1015, Q4 2SA1015, Q5 2SC1815, Q6 2SC1815, Q7 2SA1015, Q8 2SA1015, Q9 2SC1815, SW1 SW_PUSH, U1 TL082, U10 TL082, U2 LM7815CT, U3 LM7915CT, U4 TL082, U5 MN3009, U6 MN3101, U7 MN3009, U8 MN3101, U9 TL082

Commit message: KiCad version update
Other:
- net class Default removed
- net class pwr removed
